File: Hardware/B-W_Masrter/B-W_Masrter.kicad_sch (KiCad schematic)
At the start: 31 parts, among them J1 USB_C_Receptacle_USB2.0_16P, J2 Conn_02x14_Counter_Clockwise, SW1 BOOT, U1 ATmega328P-A, U2 FT232RL, U3 LM1117MP-5.0, Y1 16MHz

Commit message: docs: rewrite CLAUDE.md to match the actual design; add repo tooling
CLAUDE.md was describing a different project (ATmega32U4 / native-USB /
"Wireless Device" / WDEV-1.0 / drawing 1-20267772 / solar slave). Rewrote it
to reflect what is actually in the repo and the PM dashboard:

- Identity: Master_Slave_RF, tracking MSRF-1.0, client B-W Technology Company.
- Master (RX) board = ATmega328P + 16 MHz + CY11 433.92 MHz receiver +
  FT232RL/USB-C + onboard 5 V/600 mA mains SMPS + relay output stage.
- Only the Master board exists in the repo; Slave (TX) board not started.
- Flagged items to verify: relay coil voltage (JQC-3FF-024 = 24 V on a
  "Relay_5V"/+5 V sheet), USB-vs-SMPS power, naming/orphan-sheet cleanups.

Also add the dashboard sync tooling and project report that were untracked,
and ignore KiCad transient files (locks, autosave, backups, .kicad_prl,
fp-info-cache, *-bak), untracking the ones previously committed.

Co-Authored-By: Claude Opus 4.8 <noreply@anthropic.com>
Parts:
- removed C11, C12: 22u, Capacitor_SMD:C_0805_2012Metric_Pad1.18x1.45mm_HandSolder, symbol Device:C_Small
- removed C13, C5, C8: 100n, Capacitor_SMD:C_0402_1005Metric_Pad0.74x0.62mm_HandSolder, symbol Device:C_Small
- removed C6: 22u, Capacitor_SMD:C_0402_1005Metric_Pad0.74x0.62mm_HandSolder, symbol Device:C_Small
- removed C7: 4u7, Capacitor_SMD:C_0402_1005Metric_Pad0.74x0.62mm_HandSolder, symbol Device:C_Small
- removed D1: 1N5817M, PCM_Diode_SMD_AKL:D_MELF, symbol PCM_Diode_Schottky_AKL:1N5817M
- removed D2: USBLC6-2SC6, PCM_Package_TO_SOT_SMD_AKL:SOT-23-6, symbol PCM_Diode_TVS_AKL:USBLC6-2SC6
- removed D4: Green, LED_SMD:LED_0805_2012Metric_Pad1.15x1.40mm_HandSolder, symbol Device:LED_Small
- removed F1: Polyfuse_1A, Fuse:Fuse_1206_3216Metric_Pad1.42x1.75mm_HandSolder, symbol Device:Polyfuse_Small
- removed J1: USB_C_Receptacle_USB2.0_16P, Connector_USB:USB_C_Receptacle_GCT_USB4105-xx-A_16P_TopMnt_Horizontal, symbol Connector:USB_C_Receptacle_USB2.0_16P
- removed J2: Conn_02x14_Counter_Clockwise, symbol Connector_Generic:Conn_02x14_Counter_Clockwise
- removed R5, R6, R8: 1K, Resistor_SMD:R_0402_1005Metric_Pad0.72x0.64mm_HandSolder, symbol Device:R_Small
- removed U2: FT232RL, Package_SO:SSOP-28_5.3x10.2mm_P0.65mm, symbol Interface_USB:FT232RL
- removed U3: LM1117MP-5.0, Package_TO_SOT_SMD:SOT-223-3_TabPin2, symbol Regulator_Linear:LM1117MP-5.0
- added C1: 10u, Capacitor_SMD:C_0805_2012Metric_Pad1.18x1.45mm_HandSolder, symbol Device:C
- added C2: 22u, Capacitor_SMD:C_0805_2012Metric_Pad1.18x1.45mm_HandSolder, symbol Device:C
- added D1: BLU, LED_THT:LED_D5.0mm, symbol Device:LED
- added D2: GRN, LED_THT:LED_D5.0mm, symbol Device:LED
- added D3: YLW, LED_THT:LED_D5.0mm, symbol Device:LED
- added D4: RED, LED_THT:LED_D5.0mm, symbol Device:LED
- added J1: L, Connector_Wire:SolderWire-0.75sqmm_1x01_D1.25mm_OD3.5mm, symbol Connector:Conn_01x01_Socket
- added J2: N, Connector_Wire:SolderWire-0.75sqmm_1x01_D1.25mm_OD3.5mm, symbol Connector:Conn_01x01_Socket
- added J3, J7: Conn_01x06, Connector_PinSocket_2.54mm:PinSocket_1x06_P2.54mm_Vertical, symbol Connector_Generic:Conn_01x06
- added J4: Conn_02x06_Odd_Even, Connector_PinSocket_2.54mm:PinSocket_2x06_P2.54mm_Vertical, symbol Connector_Generic:Conn_02x06_Odd_Even
- added J5: A, Connector_Wire:SolderWire-0.75sqmm_1x01_D1.25mm_OD3.5mm, symbol Connector_Generic:Conn_01x01
- added J6: B, Connector_Wire:SolderWire-0.75sqmm_1x01_D1.25mm_OD3.5mm, symbol Connector_Generic:Conn_01x01
- added J8: Screw_Terminal_01x03, TerminalBlock_Phoenix:TerminalBlock_Phoenix_MKDS-1,5-3-5.08_1x03_P5.08mm_Horizontal, symbol Connector:Screw_Terminal_01x03
- added PS1: 5VDC, Converter_ACDC:Converte_ACDC_Module_5V_600mA, symbol Power_Supply_5V:Power_Supply_SMPS_5V600mA
- added R1: 1K, Resistor_SMD:R_0805_2012Metric_Pad1.20x1.40mm_HandSolder, symbol Device:R_Small
- added R4: 470R, Resistor_SMD:R_0805_2012Metric_Pad1.20x1.40mm_HandSolder, symbol Device:R_Small
- added U1: AMS1117-3.3, Package_TO_SOT_SMD:SOT-223-3_TabPin2, symbol Regulator_Linear:AMS1117-3.3
- added U2: CY11-CY, RF1:CY11-CY_THT, symbol CY11-CY:CY11-CY
- C3: renamed from C4; footprint Capacitor_Tantalum_SMD:CP_EIA-3216-12_Kemet-S_Pad1.58x1.35mm_HandSolder -> Capacitor_SMD:CP_Elec_4x5.4
- R2, R3: value 5K1 -> 470R; footprint Resistor_SMD:R_0402_1005Metric_Pad0.72x0.64mm_HandSolder -> Resistor_SMD:R_0805_2012Metric_Pad1.20x1.40mm_HandSolder
- renumbered C1 to C4, C2 to C5, R9 to R5, U1 to U3
Connections:
- net CC1 is gone; now on net GND: R2.1
- net CC2 is gone; now on net GND: R3.1
- net +5V: now also C1.1, D3.2 (A), J3.3 (Pin_3), U1.3 (VI)
- net A0: now also J7.1 (Pin_1)
- net A1: now also J7.2 (Pin_2)
- net A2: now also J7.3 (Pin_3)
- net A3: now also J7.4 (Pin_4)
- net A4: now also J7.5 (Pin_5)
- net A5: now also J7.6 (Pin_6)
- net AREF: now also U3.20 (AREF), J3.5 (Pin_5)
- net D10: now also J4.6 (Pin_6)
- net D2: now also D2.2 (A), J4.1 (Pin_1)
- net D3: now also J4.3 (Pin_3)
- net D4: now also D1.2 (A), J4.5 (Pin_5)
- net D5: now also D4.2 (A), J4.7 (Pin_7)
- net D6: now also J4.9 (Pin_9)
- net D7: now also J4.11 (Pin_11)
- net D8: now also J4.2 (Pin_2)
- net D9: now also J4.4 (Pin_4)
- net GND: now also C1.2, C2.2, PS1.4 (-), R1.1, R4.1, U1.1 (GND), U2.3 (GND), U2.4 (ANT); no longer R2.2, R3.2
- net RXD0: now also J3.2 (Pin_2)
- net TXD0: now also J3.1 (Pin_1)
- net ~{RESET}: now also J3.4 (Pin_4)
- net A6: no longer names the net of U3.19 (ADC6)
- net A7: no longer names the net of U3.22 (ADC7)
- net D11/MOSI renamed D11
- net D11: now also J4.10 (Pin_10), U2.2 (DT)
- net D12/MISO renamed D12
- net D12: now also J4.8 (Pin_8)
- net D13/SCK renamed D13
- net D13: now also J4.12 (Pin_12)
- new net: D3.1 (K), R3.2
- new net: D4.1 (K), R4.2
- new net: D1.1 (K), R1.2
- new net: D2.1 (K), R2.2
- new net: J1.1 (Pin_1), PS1.1 (AC/L)
- new net: J2.1 (Pin_1), PS1.2 (AC/N)
- new net +3V3: C2.1, J3.6 (Pin_6), U1.2 (VO)
- new net PROG/V_{OUT}: J5.1 (Pin_1), PS1.3 (+), U2.1 (V_{CC})
- new net Relay_5V/+5V: J6.1 (Pin_1)
- new net Relay_5V/COM: J8.2 (Pin_2)
- new net Relay_5V/NC: J8.3 (Pin_3)
- new net Relay_5V/NO: J8.1 (Pin_1)
- no-connect marks 15 -> 3
Other:
- added sheet PROG (PORG.kicad_sch)
- added sheet Relay_5V (Relay_5V.kicad_sch)
- note added: "AC_IN"
- note added: "Connectors"
- note added: "Genaral plan"
- note added: "LEDs Indicators"
- note added: "SW1"
- note added: "VOLTAGE_REGULATOR_3V3"
- note removed: "OUTPUT"
- note removed: "Polarity Reverse Protection & USB to Serial"
- note removed: "RESET"
- company: MooN_Technology -> IRAQ_PCB
- title: Arduino_Nano_DevBoard -> R_Slave
- moved on the sheet: C3, C4, C5, H1, H2, H3, H4, R5, SW1, U3, Y1
